File: andean-condor.kicad_pcb (KiCad board)
At the start: 2 copper layers, 291.8 x 129 mm, 150 parts, among them SW1 SW_SPDT

Commit message: Added some text to the pcb
Other:
- board text added: "designed by Guido Bartolucci https://github.com/guidoism/andean-condor"
Changed lines of the file:
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@@
   (gr_line (start 49.821572 109.683836) (end 63.797801 57.523842) (layer "Edge.Cuts") (width 0.15))
   (gr_line (start 66.247288 56.109629) (end 99.088767 64.909477) (layer "Edge.Cuts") (width 0.15))
+  (gr_text "designed by Guido Bartolucci\nhttps://github.com/guidoism/andean-condor" (at 195.5 134.1) (layer "B.SilkS")
+    (effects (font (size 1 1) (thickness 0.15)) (justify mirror))
+  )
   (segment (start 200.7 85.8) (end 197.1 82.2) (width 0.25) (layer "F.Cu") (net 0))
   (segment (start 197.1 82.2) (end 196.2 82.2) (width 0.25) (layer "F.Cu") (net 0))

Commit message: Checkpoint
Parts:
- removed MCU1: , ProMicro
- removed the REF** at (190.2, 85.8)
- removed the REF** at (201.9, 79.1)
- removed the REF** at (200.7, 85.8)
- removed display*: nice!view, nice_view:nice_view
- added D33: D, kbd:D3_TH_SMD_v2, F.Cu at (217.1, 89.9)
- added JST_PH2_TH: BAT, keyboard_parts:JST_PH2_TH, F.Cu at (221.2, 92.9)
- added REF**: RPi_Pico_SMD, MCU_RaspberryPi_and_Boards:RPi_Pico_SMD, F.Cu at (202.9, 104.6)
- added Ref**: Val**, kbd:M2_HOLE_v3, F.Cu at (185.8, 130.6)
- added Ref**: Val**, kbd:M2_HOLE_v3, F.Cu at (186.2, 82.7)
- added Ref**: Val**, kbd:M2_HOLE_v3, F.Cu at (219.8, 82.6)
- added Ref**: Val**, kbd:M2_HOLE_v3, F.Cu at (219.4, 130.6)
- SW1: value SW_SPDT -> PWR
- moved D42 110.6 mm to (323.1, 85.9)
- moved D60 104.0 mm to (326.7, 99.9)
- moved D40 103.8 mm to (318.1, 68.4)
- moved D44 98.6 mm to (83.8, 85.3)
- moved D41 94.7 mm to (304.7, 90.9)
- moved D49 89.8 mm to (78.7, 103.6)
- moved D37 89.4 mm to (88.0, 69.5)
- moved D59 88.0 mm to (308.0, 103.1)
- moved D39 87.9 mm to (299.4, 71.6)
- moved D43 76.7 mm to (102.1, 90.1)
- moved D33 74.9 mm to (278.3, 66.1)
- moved D50 73.4 mm to (99.2, 101.0)
- moved D38 73.3 mm to (106.5, 74.0)
- moved D43 68.9 mm to (283.1, 83.7)
- moved D48 65.9 mm to (287.2, 100.0)
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Connections:
- SW1 pad 2: RAW -> (no net)
Routing:
- net row1r: track 38.8 -> 159.9 mm, vias 0 -> 1
- net row2r: track 32.5 -> 149.4 mm
- net farpinky_home: track 119.1 -> 6.93 mm
- net mirror_farpinky_home: track 123.1 -> 12.2 mm
- net farpinky_bottom: track 112.7 -> 6.65 mm
- net mirror_farpinky_bottom: track 114.9 -> 13.7 mm
- net row3: track 35.3 -> 133.7 mm
- net mirror_farpinky_top: track 109.4 -> 12.8 mm
- net farpinky_top: track 103.9 -> 7.97 mm
- net pinky_home: track 101.1 -> 6.85 mm
- net row3r: track 35.5 -> 129.7 mm
- net mirror_pinky_home: track 104.4 -> 12.3 mm
- net row4: track 26.7 -> 116.7 mm, vias 0 -> 1
- net pinky_bottom: track 98.2 -> 11.1 mm
- net mirror_pinky_bottom: track 100.0 -> 14.4 mm
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Other:
- outline, holes or cut-outs redrawn
- board text added: "+ -"
