File: ergogen-output.2023-09-05/pcbs/andean-condor.kicad_pcb (KiCad board)
At the start: 2 copper layers, 291.8 x 129 mm, 104 parts

Commit message: Checkpoint
Parts:
- moved S25 35.4 mm to (321.0, 162.9), turned to 0 degrees
- moved S1 34.7 mm to (61.9, 93.5), turned to -30 degrees
- moved S26 34.2 mm to (321.0, 143.9), turned to 0 degrees
- moved S27 33.6 mm to (321.0, 124.9), turned to 0 degrees
- moved S2 33.5 mm to (71.4, 77.0), turned to -30 degrees
- moved S3 32.9 mm to (80.9, 60.6), turned to -30 degrees
- moved D31 32.7 mm to (312.3, 155.9), turned to -90 degrees
- moved D13 32.0 mm to (73.0, 91.8), turned to -120 degrees
- moved D19 31.9 mm to (312.3, 143.9), turned to 90 degrees
- moved D20 31.3 mm to (312.3, 124.9), turned to 90 degrees
- moved D1 31.2 mm to (79.0, 81.4), turned to 60 degrees
- moved S28 30.8 mm to (302.0, 162.9), turned to 0 degrees
- moved D2 30.6 mm to (88.5, 64.9), turned to 60 degrees
- moved S4 30.1 mm to (78.4, 103.0), turned to -30 degrees
- moved S29 29.3 mm to (302.0, 143.9), turned to 0 degrees
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Routing:
- net row2r: track 0.00 -> 108.3 mm
- net row3r: track 0.00 -> 107.2 mm
- net row1r: track 0.00 -> 107.1 mm
- net row2: track 0.00 -> 107.1 mm
- net row1: track 0.00 -> 106.8 mm
- net row3: track 0.00 -> 106.6 mm
- net mirror_index_home: track 0.00 -> 12.7 mm
- net mirror_pinky_top: track 0.00 -> 12.7 mm
- net mirror_pinky_home: track 0.00 -> 12.7 mm
- net mirror_index_top: track 0.00 -> 12.7 mm
- net mirror_ring_top: track 0.00 -> 12.7 mm
- net mirror_ring_home: track 0.00 -> 12.7 mm
- net mirror_inner_top: track 0.00 -> 12.7 mm
- net mirror_farpinky_top: track 0.00 -> 12.7 mm
- net mirror_farpinky_home: track 0.00 -> 12.7 mm
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Other:
- board size 291.8 x 129 mm -> 282 x 165.4 mm

Commit message: Checkpoint
Parts:
- moved S1 69.7 mm to (57.6, 163.1), turned to 0 degrees
- moved S25 69.4 mm to (316.7, 93.7), turned to 30 degrees
- moved S3 68.6 mm to (57.6, 125.1), turned to 0 degrees
- moved S2 68.4 mm to (57.6, 144.1), turned to 0 degrees
- moved S27 68.3 mm to (297.7, 60.8), turned to 30 degrees
- moved S26 68.1 mm to (307.2, 77.2), turned to 30 degrees
- moved D13 64.6 mm to (66.3, 156.1), turned to -90 degrees
- moved D31 64.3 mm to (305.7, 92.0), turned to -60 degrees
- moved D2 64.1 mm to (66.3, 125.1), turned to 90 degrees
- moved D1 64.0 mm to (66.3, 144.1), turned to 90 degrees
- moved D20 63.8 mm to (290.2, 65.1), turned to 120 degrees
- moved D19 63.6 mm to (299.7, 81.6), turned to 120 degrees
- moved S4 60.1 mm to (76.6, 163.1), turned to 0 degrees
- moved S28 59.8 mm to (300.2, 103.2), turned to 30 degrees
- moved S6 58.8 mm to (76.6, 125.1), turned to 0 degrees
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Routing:
- net col1: track 0.00 -> 141.2 mm
Other:
- outline, holes or cut-outs redrawn

Commit message: Checkpoint
Routing:
- net col2: track 0.00 -> 115.7 mm
Changed lines of the file:
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@@
   (segment (start 85.064326 158.006293) (end 85.334326 157.736293) (width 0.25) (layer "F.Cu") (net 5))
   (segment (start 79.174326 158.006293) (end 85.064326 158.006293) (width 0.25) (layer "F.Cu") (net 5))
+  (segment (start 72.824326 160.546294) (end 85.71731 160.546294) (width 0.25) (layer "B.Cu") (net 6))
+  (segment (start 87.213604 159.05) (end 99.213604 159.05) (width 0.25) (layer "B.Cu") (net 6))
+  (segment (start 99.213604 159.05) (end 104.613604 153.65) (width 0.25) (layer "B.Cu") (net 6))
+  (segment (start 72.824325 122.546294) (end 72.824325 141.546294) (width 0.25) (layer "B.Cu") (net 6))
+  (segment (start 72.824325 141.546294) (end 72.824326 160.546294) (width 0.25) (layer "B.Cu") (net 6))
+  (segment (start 85.71731 160.546294) (end 87.213604 159.05) (width 0.25) (layer "B.Cu") (net 6))
+  (segment (start 122.986396 153.65) (end 138.23497 168.898574) (width 0.25) (layer "B.Cu") (net 6))
+  (segment (start 138.23497 168.898574) (end 138.23497 172.010317) (width 0.25) (layer "B.Cu") (net 6))
+  (segment (start 104.613604 153.65) (end 122.986396 153.65) (width 0.25) (layer "B.Cu") (net 6))
   (segment (start 79.174326 139.006293) (end 81.904325 139.006294) (width 0.25) (layer "F.Cu") (net 7))
   (segment (start 81.904325 139.006294) (end 85.334325 142.436294) (width 0.25) (layer "F.Cu") (net 7))

Commit message: Checkpoint
Routing:
- net col3: track 0.00 -> 117.9 mm
Changed lines of the file:
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@@
   (segment (start 104.064325 146.006294) (end 104.334325 145.736294) (width 0.25) (layer "F.Cu") (net 9))
   (segment (start 98.174326 146.006294) (end 104.064325 146.006294) (width 0.25) (layer "F.Cu") (net 9))
+  (segment (start 91.824325 148.546293) (end 99.908009 148.546293) (width 0.25) (layer "B.Cu") (net 10))
+  (segment (start 91.824326 110.546293) (end 91.824327 129.546293) (width 0.25) (layer "B.Cu") (net 10))
+  (segment (start 104.561716 153.2) (end 123.172792 153.2) (width 0.25) (layer "B.Cu") (net 10))
+  (segment (start 145.772792 175.8) (end 152.713626 175.8) (width 0.25) (layer "B.Cu") (net 10))
+  (segment (start 123.172792 153.2) (end 145.772792 175.8) (width 0.25) (layer "B.Cu") (net 10))
+  (segment (start 152.713626 175.8) (end 158.191191 181.277565) (width 0.25) (layer "B.Cu") (net 10))
+  (segment (start 99.908009 148.546293) (end 104.561716 153.2) (width 0.25) (layer "B.Cu") (net 10))
+  (segment (start 91.824327 129.546293) (end 91.824327 148.546291) (width 0.25) (layer "B.Cu") (net 10))
+  (segment (start 91.824327 148.546291) (end 91.824325 148.546293) (width 0.25) (layer "B.Cu") (net 10))
   (segment (start 98.174327 127.006294) (end 100.904326 127.006293) (width 0.25) (layer "F.Cu") (net 11))
   (segment (start 100.904326 127.006293) (end 104.334325 130.436293) (width 0.25) (layer "F.Cu") (net 11))

Commit message: Checkpoint
Routing:
- net col4: track 0.00 -> 125.5 mm
Changed lines of the file:
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@@
   (segment (start 117.174325 141.006294) (end 123.064325 141.006294) (width 0.25) (layer "F.Cu") (net 13))
   (segment (start 123.064325 141.006294) (end 123.334326 140.736294) (width 0.25) (layer "F.Cu") (net 13))
+  (segment (start 110.824325 146.524325) (end 117.05 152.75) (width 0.25) (layer "B.Cu") (net 14))
+  (segment (start 155.024792 175.35) (end 175.06888 195.394088) (width 0.25) (layer "B.Cu") (net 14))
+  (segment (start 110.824327 124.546294) (end 110.824327 143.546291) (width 0.25) (layer "B.Cu") (net 14))
+  (segment (start 110.824327 143.546291) (end 110.824325 143.546293) (width 0.25) (layer "B.Cu") (net 14))
+  (segment (start 145.959188 175.35) (end 155.024792 175.35) (width 0.25) (layer "B.Cu") (net 14))
+  (segment (start 110.824325 143.546293) (end 110.824325 146.524325) (width 0.25) (layer "B.Cu") (net 14))
+  (segment (start 123.359188 152.75) (end 145.959188 175.35) (width 0.25) (layer "B.Cu") (net 14))
+  (segment (start 110.824326 105.546293) (end 110.824327 124.546294) (width 0.25) (layer "B.Cu") (net 14))
+  (segment (start 117.05 152.75) (end 123.359188 152.75) (width 0.25) (layer "B.Cu") (net 14))
   (segment (start 117.174326 122.006293) (end 119.904326 122.006293) (width 0.25) (layer "F.Cu") (net 15))
   (segment (start 119.904326 122.006293) (end 123.334325 125.436293) (width 0.25) (layer "F.Cu") (net 15))

Commit message: Checkpoint
Routing:
- net col5: track 0.00 -> 117.0 mm
- net col6: track 0.00 -> 65.4 mm
Changed lines of the file:
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@@
   (segment (start 142.064325 147.006293) (end 142.334326 146.736294) (width 0.25) (layer "F.Cu") (net 17))
   (segment (start 136.174326 147.006293) (end 142.064325 147.006293) (width 0.25) (layer "F.Cu") (net 17))
+  (segment (start 129.824325 158.578741) (end 134.872792 163.627208) (width 0.25) (layer "B.Cu") (net 18))
+  (segment (start 157.405594 177.094406) (end 183.537008 177.094406) (width 0.25) (layer "B.Cu") (net 18))
+  (segment (start 129.824325 130.546294) (end 129.824325 149.546293) (width 0.25) (layer "B.Cu") (net 18))
+  (segment (start 134.872792 163.627208) (end 143.938396 163.627208) (width 0.25) (layer "B.Cu") (net 18))
+  (segment (start 143.938396 163.627208) (end 157.405594 177.094406) (width 0.25) (layer "B.Cu") (net 18))
+  (segment (start 183.537008 177.094406) (end 189.623725 183.181123) (width 0.25) (layer "B.Cu") (net 18))
+  (segment (start 129.824326 111.546294) (end 129.824325 130.546294) (width 0.25) (layer "B.Cu") (net 18))
+  (segment (start 129.824325 149.546293) (end 129.824325 158.578741) (width 0.25) (layer "B.Cu") (net 18))
   (segment (start 136.174326 128.006294) (end 138.904327 128.006294) (width 0.25) (layer "F.Cu") (net 19))
   (segment (start 138.904327 128.006294) (end 142.334326 131.436293) (width 0.25) (layer "F.Cu") (net 19))
@@
   (segment (start 155.174326 149.006293) (end 161.064325 149.006294) (width 0.25) (layer "F.Cu") (net 21))
   (segment (start 161.064325 149.006294) (end 161.334325 148.736293) (width 0.25) (layer "F.Cu") (net 21))
+  (segment (start 148.824326 113.546293) (end 148.824327 132.546293) (width 0.25) (layer "B.Cu") (net 22))
+  (segment (start 148.824327 132.546293) (end 148.824327 151.546291) (width 0.25) (layer "B.Cu") (net 22))
+  (segment (start 148.824325 151.546293) (end 148.824325 153.626424) (width 0.25) (layer "B.Cu") (net 22))
+  (segment (start 160.911577 165.713676) (end 169.089143 165.713676) (width 0.25) (layer "B.Cu") (net 22))
+  (segment (start 148.824327 151.546291) (end 148.824325 151.546293) (width 0.25) (layer "B.Cu") (net 22))
+  (segment (start 148.824325 153.626424) (end 160.911577 165.713676) (width 0.25) (layer "B.Cu") (net 22))
   (segment (start 157.904326 130.006293) (end 161.334326 133.436293) (width 0.25) (layer "F.Cu") (net 23))
   (segment (start 155.174326 130.006293) (end 157.904326 130.006293) (width 0.25) (layer "F.Cu") (net 23))

Commit message: Checkpoint
Parts:
- moved S1 35.7 mm to (53.7, 127.6), turned to -15 degrees
- moved S2 34.8 mm to (58.7, 109.3), turned to -15 degrees
- moved S3 34.7 mm to (63.6, 90.9), turned to -15 degrees
- moved S25 34.3 mm to (321.9, 127.6), turned to 15 degrees
- moved S26 33.5 mm to (317.0, 109.3), turned to 15 degrees
- moved S27 33.4 mm to (312.1, 90.9), turned to 15 degrees
- moved D13 33.1 mm to (64.0, 123.1), turned to -105 degrees
- moved D1 32.6 mm to (67.1, 111.5), turned to 75 degrees
- moved D2 32.4 mm to (72.0, 93.2), turned to 75 degrees
- moved D31 31.7 mm to (311.7, 123.1), turned to -75 degrees
- moved D19 31.3 mm to (308.6, 111.5), turned to 105 degrees
- moved D20 31.1 mm to (303.7, 93.2), turned to 105 degrees
- moved S4 30.9 mm to (72.1, 132.5), turned to -15 degrees
- moved S5 29.9 mm to (77.0, 114.2), turned to -15 degrees
- moved S6 29.7 mm to (81.9, 95.8), turned to -15 degrees
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Routing:
- net col4: track 125.5 -> 254.0 mm
- net col1: track 141.2 -> 262.9 mm
- net col5: track 117.0 -> 238.1 mm
- net col3: track 117.9 -> 238.0 mm
- net col2: track 115.7 -> 233.7 mm
- net col6: track 65.4 -> 131.7 mm
- net row3r: track 107.2 -> 148.2 mm
- net row2r: track 108.3 -> 148.4 mm
- net row3: track 106.6 -> 146.5 mm
- net row1r: track 107.1 -> 138.7 mm
- net row2: track 107.1 -> 129.3 mm
- net row1: track 106.8 -> 125.3 mm
Other:
- board size 282 x 165.4 mm -> 291.8 x 129 mm

Commit message: Checkpoint
Routing:
- net col5: track 238.1 -> 298.4 mm
- net col6: track 131.7 -> 186.1 mm
- net col2: track 233.7 -> 270.7 mm
- net col4: track 254.0 -> 291.0 mm
- net col3: track 238.0 -> 275.0 mm
- net col1: track 262.9 -> 297.9 mm
Changed lines of the file:
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@@
   (segment (start 63.196664 124.890292) (end 63.527346 124.699374) (width 0.25) (layer "F.Cu") (net 1))
   (segment (start 57.50736 123.365849) (end 63.196664 124.890292) (width 0.25) (layer "F.Cu") (net 1))
+  (segment (start 171 173) (end 206 173) (width 0.25) (layer "F.Cu") (net 2))
   (segment (start 76.867038 137.760701) (end 53.199827 131.419091) (width 0.25) (layer "B.Cu") (net 2))
   (segment (start 257.532568 136.658893) (end 273.439736 132.396581) (width 0.25) (layer "B.Cu") (net 2))
@@
   (segment (start 81.549255 129.807854) (end 81.879937 129.616936) (width 0.25) (layer "F.Cu") (net 5))
   (segment (start 75.859952 128.28341) (end 81.549255 129.807854) (width 0.25) (layer "F.Cu") (net 5))
+  (segment (start 170 172) (end 207 172) (width 0.25) (layer "F.Cu") (net 6))
   (segment (start 289.949606 96.36595) (end 289.949604 96.365948) (width 0.25) (layer "B.Cu") (net 6))
   (segment (start 253.560246 153.252416) (end 252.499586 155.089534) (width 0.25) (layer "B.Cu") (net 6))
@@
   (segment (start 103.007673 123.134307) (end 103.338354 122.943388) (width 0.25) (layer "F.Cu") (net 9))
   (segment (start 97.318371 121.609863) (end 103.007673 123.134307) (width 0.25) (layer "F.Cu") (net 9))
+  (segment (start 170 171) (end 207 171) (width 0.25) (layer "F.Cu") (net 10))
   (segment (start 272.871357 106.039425) (end 277.788918 124.392013) (width 0.25) (layer "B.Cu") (net 10))
   (segment (start 253.731227 136.745711) (end 243.593151 154.305374) (width 0.25) (layer "B.Cu") (net 10))
@@
   (segment (start 116.965056 121.697796) (end 122.654359 123.22224) (width 0.25) (layer "F.Cu") (net 13))
   (segment (start 122.654359 123.22224) (end 122.985042 123.031321) (width 0.25) (layer "F.Cu") (net 13))
+  (segment (start 170 170) (end 207 170) (width 0.25) (layer "F.Cu") (net 14))
   (segment (start 109.403255 125.384303) (end 113.805473 133.009166) (width 0.25) (layer "B.Cu") (net 14))
   (segment (start 216.031534 191.101152) (end 213.483157 195.51507) (width 0.25) (layer "B.Cu") (net 14))
@@
   (segment (start 139.454036 133.935356) (end 139.784718 133.744438) (width 0.25) (layer "F.Cu") (net 17))
   (segment (start 133.764734 132.410912) (end 139.454036 133.935356) (width 0.25) (layer "F.Cu") (net 17))
+  (segment (start 192.71004 188.092903) (end 196.426111 188.092903) (width 0.25) (layer "F.Cu") (net 18))
+  (segment (start 185.803973 181.186836) (end 192.71004 188.092903) (width 0.25) (layer "F.Cu") (net 18))
+  (segment (start 176.030153 181.186836) (end 185.803973 181.186836) (width 0.25) (layer "F.Cu") (net 18))
+  (segment (start 170 169) (end 207 169) (width 0.25) (layer "F.Cu") (net 18))
   (segment (start 243.000125 153.532527) (end 231.149942 156.707774) (width 0.25) (layer "B.Cu") (net 18))
   (segment (start 241.342556 135.193064) (end 245.224339 149.680074) (width 0.25) (layer "B.Cu") (net 18))
@@
   (segment (start 151.599687 139.260325) (end 157.288988 140.78477) (width 0.25) (layer "F.Cu") (net 21))
   (segment (start 157.288988 140.78477) (end 157.61967 140.59385) (width 0.25) (layer "F.Cu") (net 21))
+  (segment (start 169.815987 168.099646) (end 206.799846 168.099646) (width 0.25) (layer "F.Cu") (net 22))
+  (segment (start 206.799846 168.099646) (end 210.062396 164.837096) (width 0.25) (layer "F.Cu") (net 22))
+  (segment (start 160.716178 158.999837) (end 169.815987 168.099646) (width 0.25) (layer "F.Cu") (net 22))
   (segment (start 154.643781 103.365094) (end 149.726219 121.717685) (width 0.25) (layer "B.Cu") (net 22))
   (segment (start 213.67248 105.337296) (end 218.590043 123.689887) (width 0.25) (layer "B.Cu") (net 22))
