File: ergogen-output.2023-09-05/pcbs/andean-condor.kicad_pcb (KiCad board)
At the start: 2 copper layers, 291.8 x 129 mm, 104 parts

Commit message: Checkpoint
Routing:
- net row4: track 0.00 -> 193.1 mm, vias 0 -> 5
- net col1: track 297.9 -> 434.5 mm, vias 0 -> 2
- net row4r: track 0.00 -> 86.5 mm, vias 0 -> 1
- net col2: track 270.7 -> 330.4 mm
- net col6: track 186.1 -> 227.9 mm, vias 0 -> 1
- net col3: track 275.0 -> 299.0 mm
- net col4: track 291.0 -> 310.3 mm, vias 0 -> 2
- net col5: track 298.4 -> 297.1 mm, vias 0 -> 3

Commit message: Checkpoint
Routing:
- net GND: track 0.00 -> 99.6 mm, vias 0 -> 5
- net switch_from: track 0.00 -> 59.5 mm, vias 0 -> 2
- net SDA: track 0.00 -> 56.9 mm, vias 0 -> 2
- net col4: track 310.3 -> 362.4 mm, vias 2 -> 3
- net CS: track 0.00 -> 50.8 mm
- net col5: track 297.1 -> 345.2 mm, vias 3 -> 4
- net col3: track 299.0 -> 346.0 mm, vias 0 -> 1
- net RST: track 0.00 -> 45.4 mm, vias 0 -> 3
- net col2: track 330.4 -> 375.5 mm, vias 0 -> 1
- net VCC: track 0.00 -> 32.6 mm, vias 0 -> 1
- net SCL: track 0.00 -> 30.0 mm, vias 0 -> 1
- net RAW: track 0.00 -> 7.94 mm

Commit message: Checkpoint
Parts:
- moved B1 3.08 mm to (190.9, 145.8)
- moved D18 3.08 mm to (161.1, 139.2)
- moved D24 3.08 mm to (267.0, 91.6)
- moved D31 3.08 mm to (314.8, 123.3)
- moved S13 3.08 mm to (133.1, 136.8)
- moved S46 3.08 mm to (217.5, 163.7)
- moved D11 3.08 mm to (164.2, 127.6)
- moved D20 3.08 mm to (306.8, 93.3)
- moved D21 3.08 mm to (293.3, 116.6)
- moved D22 3.08 mm to (288.4, 98.3)
- moved D25 3.08 mm to (252.2, 110.0)
- moved D26 3.08 mm to (247.3, 91.7)
- moved D27 3.08 mm to (235.4, 120.7)
- moved D33 3.08 mm to (275.0, 121.5)
- moved S25 3.08 mm to (325.0, 127.8)
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Routing:
- net row4r: track 86.5 -> 183.9 mm, vias 1 -> 3
- net col1: track 434.5 -> 499.0 mm
- net col2: track 375.5 -> 418.5 mm
- net col3: track 346.0 -> 372.4 mm, vias 1 -> 2
- net col4: track 362.4 -> 384.3 mm, vias 3 -> 4

Commit message: Checkpoint
Routing:
- net col5: track 345.2 -> 121.1 mm, vias 4 -> 0

Commit message: Checkpoint
Parts:
- moved S31 60.5 mm to (312.4, 72.0)
- moved D23 60.5 mm to (299.1, 55.9)
- moved S17 60.5 mm to (183.0, 71.3)
- moved D2 60.5 mm to (102.2, 39.3)
- moved D5 60.5 mm to (137.1, 55.9)
- moved S24 60.5 mm to (205.6, 131.8)
- moved D26 60.5 mm to (274.5, 37.6)
- moved S40 60.5 mm to (258.1, 89.6)
- moved D38 60.5 mm to (170.3, 103.2)
- moved D40 60.5 mm to (201.4, 107.9)
- moved D45 60.5 mm to (249.4, 120.1)
- moved S16 60.5 mm to (178.1, 89.6)
- moved S23 60.5 mm to (188.4, 139.8)
- moved S26 60.5 mm to (347.3, 55.4)
- moved S30 60.5 mm to (324.0, 41.9)
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Routing:
- net col5: track 121.1 -> 299.8 mm, vias 0 -> 3

Commit message: Checkpoint
Routing:
- net col5: track 299.8 -> 347.8 mm, vias 3 -> 4
Changed lines of the file:
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@@
   (segment (start 169.71149 80.032824) (end 170.042171 79.841907) (width 0.25) (layer "F.Cu") (net 17))
   (segment (start 164.022188 78.50838) (end 169.71149 80.032824) (width 0.25) (layer "F.Cu") (net 17))
+  (segment (start 229.673505 115.073505) (end 229.7 115.1) (width 0.25) (layer "F.Cu") (net 18))
   (segment (start 250.307646 115.073505) (end 255.881151 109.5) (width 0.25) (layer "F.Cu") (net 18))
   (segment (start 255.881151 109.5) (end 257.6 109.5) (width 0.25) (layer "F.Cu") (net 18))
   (segment (start 178.976651 115.073505) (end 206.226495 115.073505) (width 0.25) (layer "F.Cu") (net 18))
   (segment (start 206.226495 115.073505) (end 206.3 115) (width 0.25) (layer "F.Cu") (net 18))
-  (segment (start 206.373505 115.073505) (end 250.307646 115.073505) (width 0.25) (layer "F.Cu") (net 18))
+  (segment (start 206.373505 115.073505) (end 229.673505 115.073505) (width 0.25) (layer "F.Cu") (net 18))
+  (segment (start 229.7 115.1) (end 229.726495 115.073505) (width 0.25) (layer "F.Cu") (net 18))
   (segment (start 206.3 115) (end 206.373505 115.073505) (width 0.25) (layer "F.Cu") (net 18))
+  (segment (start 229.726495 115.073505) (end 250.307646 115.073505) (width 0.25) (layer "F.Cu") (net 18))
   (via (at 257.6 109.5) (size 0.8) (drill 0.4) (layers "F.Cu" "B.Cu") (net 18))
+  (via (at 229.7 115.1) (size 0.8) (drill 0.4) (layers "F.Cu" "B.Cu") (net 18))
   (via (at 206.3 115) (size 0.8) (drill 0.4) (layers "F.Cu" "B.Cu") (net 18))
   (via (at 178.976651 115.073505) (size 0.8) (drill 0.4) (layers "F.Cu" "B.Cu") (net 18))
@@
   (segment (start 162.148718 60.965741) (end 157.231157 79.318331) (width 0.25) (layer "B.Cu") (net 18))
   (segment (start 261.764887 44.58535) (end 266.682449 62.93794) (width 0.25) (layer "B.Cu") (net 18))
+  (segment (start 225.715759 68.712115) (end 229.7 72.696356) (width 0.25) (layer "B.Cu") (net 18))
+  (segment (start 229.7 72.696356) (end 229.7 115) (width 0.25) (layer "B.Cu") (net 18))
   (segment (start 167.066281 42.613149) (end 162.148718 60.965741) (width 0.25) (layer "B.Cu") (net 18))
   (segment (start 271.600009 81.29053) (end 271.600009 81.290533) (width 0.25) (layer "B.Cu") (net 18))

Commit message: Checkpoint
Connections:
- ? pad 1: (no net) -> SCL
- ? pad 1: (no net) -> VCC
Routing:
- net GND: track 99.6 -> 116.7 mm
- net extra1: track 0.00 -> 14.6 mm
- net CS: track 50.8 -> 65.4 mm
- net SCL: track 30.0 -> 43.4 mm
- net SDA: track 56.8 -> 70.2 mm
- net VCC: track 32.5 -> 44.9 mm
- net RST: track 45.4 -> 57.7 mm
- net row1: track 125.3 -> 127.9 mm

Commit message: Checkpoint
Connections:
- ? pad 1: SCL -> switch_from
Routing:
- net switch_from: track 59.4 -> 70.3 mm
- net col1: track 498.9 -> 502.6 mm
- net col2: track 418.5 -> 419.3 mm
Other:
- outline, holes or cut-outs redrawn
- board text added: "Andean Condor by Guido Bartolucci"
- board text added: "JLCJLCJLCJLC"
